File: Pivot_stand.kicad_sch (KiCad schematic)
At the start: 11 parts, among them J1 USB_B_Micro, J2 Conn_01x02_Male, U1 IFX27001TFV33

Commit message: Changed footprint library
Changed footprint library to use the BadgePirtate library
Parts:
- C1: footprint Capacitor_SMD:C_0805_2012Metric -> BadgePirates:C_0805_2012Metric
- C2, C3: footprint Capacitor_SMD:C_0805_2012Metric_Pad1.18x1.45mm_HandSolder -> BadgePirates:C_0805_2012Metric
- R1, R2, R3: footprint Resistor_SMD:R_1206_3216Metric -> BadgePirates:R_1206_3216Metric
- R4: footprint Resistor_SMD:R_0603_1608Metric_Pad1.05x0.95mm_HandSolder -> BadgePirates:R_1206_3216Metric
- U1: footprint BadgePiratesFootprint:SOT-223 -> BadgePirates:SOT-223
Changed lines of the file:
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@@
       (effects (font (size 1.27 1.27)) (justify left))
     )
-    (property "Footprint" "Capacitor_SMD:C_0805_2012Metric" (id 2) (at 167.64 72.39 0)
+    (property "Footprint" "BadgePirates:C_0805_2012Metric" (id 2) (at 167.64 72.39 0)
       (effects (font (size 1.27 1.27)) hide)
     )
@@
       (effects (font (size 1.27 1.27)) (justify left))
     )
-    (property "Footprint" "Resistor_SMD:R_1206_3216Metric" (id 2) (at 178.562 72.39 90)
+    (property "Footprint" "BadgePirates:R_1206_3216Metric" (id 2) (at 178.562 72.39 90)
       (effects (font (size 1.27 1.27)) hide)
     )
@@
       (effects (font (size 1.27 1.27)) (justify left))
     )
-    (property "Footprint" "Resistor_SMD:R_1206_3216Metric" (id 2) (at 151.892 88.9 90)
+    (property "Footprint" "BadgePirates:R_1206_3216Metric" (id 2) (at 151.892 88.9 90)
       (effects (font (size 1.27 1.27)) hide)
     )
@@
       (effects (font (size 1.27 1.27)) (justify left))
     )
-    (property "Footprint" "Resistor_SMD:R_1206_3216Metric" (id 2) (at 190.5 70.358 90)
+    (property "Footprint" "BadgePirates:R_1206_3216Metric" (id 2) (at 190.5 70.358 90)
       (effects (font (size 1.27 1.27)) hide)
     )
@@
       (effects (font (size 1.27 1.27)) (justify left))
     )
-    (property "Footprint" "Resistor_SMD:R_0603_1608Metric_Pad1.05x0.95mm_HandSolder" (id 2) (at 103.632 86.36 90)
+    (property "Footprint" "BadgePirates:R_1206_3216Metric" (id 2) (at 103.632 86.36 90)
       (effects (font (size 1.27 1.27)) hide)
     )
@@
       (effects (font (size 1.27 1.27)) (justify left))
     )
-    (property "Footprint" "Capacitor_SMD:C_0805_2012Metric_Pad1.18x1.45mm_HandSolder" (id 2) (at 96.2152 90.17 0)
+    (property "Footprint" "BadgePirates:C_0805_2012Metric" (id 2) (at 96.2152 90.17 0)
       (effects (font (size 1.27 1.27)) hide)
     )
@@
       (effects (font (size 1.27 1.27)) (justify left))
     )
-    (property "Footprint" "Capacitor_SMD:C_0805_2012Metric_Pad1.18x1.45mm_HandSolder" (id 2) (at 141.9352 82.55 0)
+    (property "Footprint" "BadgePirates:C_0805_2012Metric" (id 2) (at 141.9352 82.55 0)
       (effects (font (size 1.27 1.27)) hide)
     )
@@
     (property "Reference" "U1" (id 0) (at 153.67 62.3402 0))
     (property "Value" "IFX27001TFV33" (id 1) (at 153.67 64.8771 0))
-    (property "Footprint" "BadgePiratesFootprint:SOT-223" (id 2) (at 153.67 69.85 0)
+    (property "Footprint" "BadgePirates:SOT-223" (id 2) (at 153.67 69.85 0)
       (effects (font (size 1.27 1.27)) hide)
     )
@@
     )
     (path "/00000000-0000-0000-0000-000060e4098a"
-      (reference "C1") (unit 1) (value "10uF") (footprint "Capacitor_SMD:C_0805_2012Metric")
+      (reference "C1") (unit 1) (value "10uF") (footprint "BadgePirates:C_0805_2012Metric")
     )
     (path "/00000000-0000-0000-0000-0000634cfdf9"
-      (reference "C2") (unit 1) (value "0.1uF") (footprint "Capacitor_SMD:C_0805_2012Metric_Pad1.18x1.45mm_HandSolder")
+      (reference "C2") (unit 1) (value "0.1uF") (footprint "BadgePirates:C_0805_2012Metric")
     )
     (path "/00000000-0000-0000-0000-0000634d2767"
-      (reference "C3") (unit 1) (value "0.1uF") (footprint "Capacitor_SMD:C_0805_2012Metric_Pad1.18x1.45mm_HandSolder")
+      (reference "C3") (unit 1) (value "0.1uF") (footprint "BadgePirates:C_0805_2012Metric")
     )
     (path "/00000000-0000-0000-0000-000060fab1c6"
@@
     )
     (path "/00000000-0000-0000-0000-000060e419b2"
-      (reference "R1") (unit 1) (value "R") (footprint "Resistor_SMD:R_1206_3216Metric")
+      (reference "R1") (unit 1) (value "R") (footprint "BadgePirates:R_1206_3216Metric")
     )
     (path "/00000000-0000-0000-0000-0000634c8f07"
-      (reference "R2") (unit 1) (value "0") (footprint "Resistor_SMD:R_1206_3216Metric")
+      (reference "R2") (unit 1) (value "0") (footprint "BadgePirates:R_1206_3216Metric")
     )
     (path "/00000000-0000-0000-0000-0000634ce49d"
-      (reference "R3") (unit 1) (value "0") (footprint "Resistor_SMD:R_1206_3216Metric")
+      (reference "R3") (unit 1) (value "0") (footprint "BadgePirates:R_1206_3216Metric")
     )
     (path "/00000000-0000-0000-0000-0000634cf86b"
-      (reference "R4") (unit 1) (value "1M") (footprint "Resistor_SMD:R_0603_1608Metric_Pad1.05x0.95mm_HandSolder")
+      (reference "R4") (unit 1) (value "1M") (footprint "BadgePirates:R_1206_3216Metric")
     )
     (path "/27f176fa-5907-47fa-b2d2-85c41dd0f18b"
-      (reference "U1") (unit 1) (value "IFX27001TFV33") (footprint "BadgePiratesFootprint:SOT-223")
-    )
-  )
+      (reference "U1") (unit 1) (value "IFX27001TFV33") (footprint "BadgePirates:SOT-223")
+    )
+  )

Commit message: Change SW1 footprint
Changed SW1 footprint to use the BP lib
Parts:
- I/O1: footprint Button_Switch_SMD:SW_SPDT_CK-JS102011SAQN -> BadgePirates:SW_SPDT_PCM12
Changed lines of the file:
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@@
     (property "Reference" "I/O1" (id 0) (at 134.62 58.801 0))
     (property "Value" "SW_DPDT_x2" (id 1) (at 134.62 61.1124 0))
-    (property "Footprint" "Button_Switch_SMD:SW_SPDT_CK-JS102011SAQN" (id 2) (at 134.62 66.04 0)
+    (property "Footprint" "BadgePirates:SW_SPDT_PCM12" (id 2) (at 134.62 66.04 0)
       (effects (font (size 1.27 1.27)) hide)
     )
@@
     )
     (path "/00000000-0000-0000-0000-000060fab1c6"
-      (reference "I/O1") (unit 1) (value "SW_DPDT_x2") (footprint "Button_Switch_SMD:SW_SPDT_CK-JS102011SAQN")
+      (reference "I/O1") (unit 1) (value "SW_DPDT_x2") (footprint "BadgePirates:SW_SPDT_PCM12")
     )
     (path "/00000000-0000-0000-0000-000060e39c54"

Commit message: Fixed ref des
Fixed I/O ref des
Parts:
- renumbered I/O1 to I/O
Changed lines of the file:
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@@
   (symbol (lib_id "Switch:SW_DPDT_x2") (at 134.62 66.04 0) (unit 1)
     (in_bom yes) (on_board yes)
-    (property "Reference" "I/O1" (id 0) (at 134.62 58.801 0))
+    (property "Reference" "I/O" (id 0) (at 134.62 58.801 0))
     (property "Value" "SW_DPDT_x2" (id 1) (at 134.62 61.1124 0))
     (property "Footprint" "BadgePirates:SW_SPDT_PCM12" (id 2) (at 134.62 66.04 0)
@@
     )
     (path "/00000000-0000-0000-0000-000060fab1c6"
-      (reference "I/O1") (unit 1) (value "SW_DPDT_x2") (footprint "BadgePirates:SW_SPDT_PCM12")
+      (reference "I/O") (unit 1) (value "SW_DPDT_x2") (footprint "BadgePirates:SW_SPDT_PCM12")
     )
     (path "/00000000-0000-0000-0000-000060e39c54"

Commit message: Layout updates
Added new parts to PCB to match schematic changes.
Parts:
- renumbered I/O to I/O1
Connections:
- net ADJ: now reaches R1.2, R2.1, U1.1 (GND)
Changed lines of the file:
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@@
     (stroke (width 0) (type default) (color 0 0 0 0))
+  )
+  (label "ADJ" (at 160.02 83.82 0)
+    (effects (font (size 1.27 1.27)) (justify left bottom))
   )
   (symbol (lib_id "Pivot_stand-rescue:USB_B_Micro-Connector") (at 113.03 71.12 0) (unit 1)
@@
   (symbol (lib_id "Switch:SW_DPDT_x2") (at 134.62 66.04 0) (unit 1)
     (in_bom yes) (on_board yes)
-    (property "Reference" "I/O" (id 0) (at 134.62 58.801 0))
+    (property "Reference" "I/O1" (id 0) (at 134.62 58.801 0))
     (property "Value" "SW_DPDT_x2" (id 1) (at 134.62 61.1124 0))
     (property "Footprint" "BadgePirates:SW_SPDT_PCM12" (id 2) (at 134.62 66.04 0)
@@
     )
     (path "/00000000-0000-0000-0000-000060fab1c6"
-      (reference "I/O") (unit 1) (value "SW_DPDT_x2") (footprint "BadgePirates:SW_SPDT_PCM12")
+      (reference "I/O1") (unit 1) (value "SW_DPDT_x2") (footprint "BadgePirates:SW_SPDT_PCM12")
     )
     (path "/00000000-0000-0000-0000-000060e39c54"
